Commit message: Gripper

File: src/ur10_description/urdf/ur10_gz.urdf.xacro (robot description, xacro)
@@ -34,4 +34,11 @@
   <xacro:include filename="$(find ur10_description)/urdf/ur10_wrist_camera_gz.xacro"/>
   <xacro:ur10_wrist_camera_gz tf_prefix="$(arg tf_prefix)"/>
+  <!-- Robotiq 2F-85 gripper on tool0: UR adapter + gripper macro (control in ur10_ros2_control_gz.xacro) -->
+  <xacro:include filename="$(find robotiq_description)/urdf/ur_to_robotiq_adapter.urdf.xacro"/>
+  <xacro:include filename="$(find robotiq_description)/urdf/robotiq_2f_85_macro.urdf.xacro"/>
+  <xacro:ur_to_robotiq prefix="$(arg tf_prefix)" parent="$(arg tf_prefix)tool0" child="$(arg tf_prefix)robotiq_85_adapter_mount"/>
+  <xacro:robotiq_gripper name="RobotiqGripper" prefix="$(arg tf_prefix)" parent="$(arg tf_prefix)robotiq_85_adapter_mount" sim_gazebo="true" include_ros2_control="false">
+    <origin xyz="0 0 0" rpy="0 0 0"/>
+  </xacro:robotiq_gripper>
   <!-- Pass controllers path via property (xacro:include ignores child elements) -->
   <xacro:property name="controllers_file" value="$(find ur10_gz_bringup)/config/controllers.yaml"/>

File: src/ur10_description/urdf/ur10_ros2_control_gz.xacro (robot description, xacro)
@@ -37,4 +37,9 @@
       <state_interface name="velocity"/>
     </joint>
+    <joint name="robotiq_85_left_knuckle_joint">
+      <command_interface name="position"/>
+      <state_interface name="position"/>
+      <state_interface name="velocity"/>
+    </joint>
   </ros2_control>
   <gazebo>

Commit message: revert first gripper

File: src/ur10_description/urdf/ur10_gz.urdf.xacro (robot description, xacro)
@@ -34,11 +34,4 @@
   <xacro:include filename="$(find ur10_description)/urdf/ur10_wrist_camera_gz.xacro"/>
   <xacro:ur10_wrist_camera_gz tf_prefix="$(arg tf_prefix)"/>
-  <!-- Robotiq 2F-85 gripper on tool0: UR adapter + gripper macro (control in ur10_ros2_control_gz.xacro) -->
-  <xacro:include filename="$(find robotiq_description)/urdf/ur_to_robotiq_adapter.urdf.xacro"/>
-  <xacro:include filename="$(find robotiq_description)/urdf/robotiq_2f_85_macro.urdf.xacro"/>
-  <xacro:ur_to_robotiq prefix="$(arg tf_prefix)" parent="$(arg tf_prefix)tool0" child="$(arg tf_prefix)robotiq_85_adapter_mount"/>
-  <xacro:robotiq_gripper name="RobotiqGripper" prefix="$(arg tf_prefix)" parent="$(arg tf_prefix)robotiq_85_adapter_mount" sim_gazebo="true" include_ros2_control="false">
-    <origin xyz="0 0 0" rpy="0 0 0"/>
-  </xacro:robotiq_gripper>
   <!-- Pass controllers path via property (xacro:include ignores child elements) -->
   <xacro:property name="controllers_file" value="$(find ur10_gz_bringup)/config/controllers.yaml"/>

File: src/ur10_description/urdf/ur10_ros2_control_gz.xacro (robot description, xacro)
@@ -37,9 +37,4 @@
       <state_interface name="velocity"/>
     </joint>
-    <joint name="robotiq_85_left_knuckle_joint">
-      <command_interface name="position"/>
-      <state_interface name="position"/>
-      <state_interface name="velocity"/>
-    </joint>
   </ros2_control>
   <gazebo>

File: src/ur10_description/urdf/ur10_wrist_camera_gz.xacro (robot description, xacro)
@@ -32,5 +32,5 @@
     <parent link="${tf_prefix}tool0"/>
     <child link="${tf_prefix}wrist_camera_link"/>
-    <origin xyz="0 0 0.02" rpy="0 -1.5708 0"/>
+    <origin xyz="0 0.2 0.02" rpy="0 -1.5708 0"/>
   </joint>
   <!-- Prevent lumping so wrist_camera_link exists in Gazebo and topic path is predictable -->
